File: ressources/gazpar-kicad/Gazpar.kicad_sch (KiCad schematic)
At the start: 7 parts, among them U1 PC817, U2 ESP32-DEVKITC-32D

Commit message: Monocouche, fichiers de production, kibot, nomenclature, ...
Parts:
- added H1, H2, H3, H4: MountingHole_2.5mm_Pad_TopOnly, MountingHole:MountingHole_2.5mm_Pad_TopOnly, symbol Mechanical:MountingHole
- D1: manf (none) -> ONSEMI; manf# (none) -> 1N4148TR
- D2: manf (none) -> BROADCOM; manf# (none) -> HLMP-Y301-F0000
- Gazpar1: S1MN (none) -> AMPHENOL; S1PN (none) -> VI0221550000G; manf (none) -> CAMDENBOSS; manf# (none) -> CTBP0108/2
- R1: value 330 -> 330Ω; manf (none) -> YAGEO; manf# (none) -> CFR-25JR-52-330R
- R2: value 1k -> 1kΩ; manf (none) -> YAGEO; manf# (none) -> CFR-25JB-52-1K
- U1: manf (none) -> BROADCOM; manf# (none) -> HCPL-817-000E
- U2: footprint MODULE_ESP32-DEVKITC-32D -> ESP32-DEVKITC-32D:MODULE_ESP32-DEVKITC-32D; manf (none) -> CONNFLY;CONNFLY; manf# (none) -> DS1002-01-1*19V13;DS1002-01-1*19V13
Changed lines of the file:
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@@
       (effects (font (size 1.27 1.27)) hide)
     )
-    (pin "1")
-    (pin "2")
+    (property "manf" "BROADCOM" (id 4) (at 87.63 80.01 0)
+      (effects (font (size 1.27 1.27)) hide)
+    )
+    (property "manf#" "HLMP-Y301-F0000" (id 5) (at 87.63 80.01 0)
+      (effects (font (size 1.27 1.27)) hide)
+    )
+    (pin "1")
+    (pin "2")
+  )
+  (symbol (lib_id "Mechanical:MountingHole") (at 29.845 127.635 0) (unit 1)
+    (in_bom no) (on_board yes) (fields_autoplaced)
+    (property "Reference" "H4" (id 0) (at 32.385 126.8003 0)
+      (effects (font (size 1.27 1.27)) (justify left))
+    )
+    (property "Value" "MountingHole_2.5mm_Pad_TopOnly" (id 1) (at 32.385 129.3372 0)
+      (effects (font (size 1.27 1.27)) (justify left))
+    )
+    (property "Footprint" "MountingHole:MountingHole_2.5mm_Pad_TopOnly" (id 2) (at 29.845 127.635 0)
+      (effects (font (size 1.27 1.27)) hide)
+    )
+    (property "Datasheet" "~" (id 3) (at 29.845 127.635 0)
+      (effects (font (size 1.27 1.27)) hide)
+    )
   )
   (symbol (lib_id "ESP32-DEVKITC-32D:ESP32-DEVKITC-32D") (at 129.54 60.96 0) (unit 1)
@@
     (property "Reference" "U2" (id 0) (at 129.54 30.48 0))
     (property "Value" "ESP32-DEVKITC-32D" (id 1) (at 129.54 33.02 0))
-    (property "Footprint" "MODULE_ESP32-DEVKITC-32D" (id 2) (at 129.54 60.96 0)
+    (property "Footprint" "ESP32-DEVKITC-32D:MODULE_ESP32-DEVKITC-32D" (id 2) (at 129.54 60.96 0)
       (effects (font (size 1.27 1.27)) (justify left bottom) hide)
     )
@@
     (property "PARTREV" "4" (id 5) (at 129.54 60.96 0)
       (effects (font (size 1.27 1.27)) (justify left bottom) hide)
+    )
+    (property "manf" "CONNFLY;CONNFLY" (id 6) (at 129.54 60.96 0)
+      (effects (font (size 1.27 1.27)) hide)
+    )
+    (property "manf#" "DS1002-01-1*19V13;DS1002-01-1*19V13" (id 7) (at 129.54 60.96 0)
+      (effects (font (size 1.27 1.27)) hide)
     )
     (pin "1")
@@
     (pin "9")
   )
+  (symbol (lib_id "Mechanical:MountingHole") (at 29.845 109.22 0) (unit 1)
+    (in_bom no) (on_board yes) (fields_autoplaced)
+    (property "Reference" "H1" (id 0) (at 32.385 108.3853 0)
+      (effects (font (size 1.27 1.27)) (justify left))
+    )
+    (property "Value" "MountingHole_2.5mm_Pad_TopOnly" (id 1) (at 32.385 110.9222 0)
+      (effects (font (size 1.27 1.27)) (justify left))
+    )
+    (property "Footprint" "MountingHole:MountingHole_2.5mm_Pad_TopOnly" (id 2) (at 29.845 109.22 0)
+      (effects (font (size 1.27 1.27)) hide)
+    )
+    (property "Datasheet" "~" (id 3) (at 29.845 109.22 0)
+      (effects (font (size 1.27 1.27)) hide)
+    )
+  )
   (symbol (lib_id "Diode:1N4148") (at 66.04 87.63 270) (unit 1)
     (in_bom yes) (on_board yes) (fields_autoplaced)
@@
       (effects (font (size 1.27 1.27)) hide)
     )
+    (property "manf" "ONSEMI" (id 4) (at 66.04 87.63 0)
+      (effects (font (size 1.27 1.27)) hide)
+    )
+    (property "manf#" "1N4148TR" (id 5) (at 66.04 87.63 0)
+      (effects (font (size 1.27 1.27)) hide)
+    )
     (pin "1")
     (pin "2")
@@
     (in_bom yes) (on_board yes) (fields_autoplaced)
     (property "Reference" "R2" (id 0) (at 73.66 73.66 90))
-    (property "Value" "1k" (id 1) (at 73.66 76.2 90))
+    (property "Value" "1kΩ" (id 1) (at 73.66 76.2 90))
     (property "Footprint" "Resistor_THT:R_Axial_DIN0207_L6.3mm_D2.5mm_P7.62mm_Horizontal" (id 2) (at 73.66 78.232 90)
       (effects (font (size 1.27 1.27)) hide)
     )
     (property "Datasheet" "~" (id 3) (at 73.66 80.01 0)
+      (effects (font (size 1.27 1.27)) hide)
+    )
+    (property "manf" "YAGEO" (id 4) (at 73.66 80.01 0)
+      (effects (font (size 1.27 1.27)) hide)
+    )
+    (property "manf#" "CFR-25JB-52-1K" (id 5) (at 73.66 80.01 0)
       (effects (font (size 1.27 1.27)) hide)
     )
@@
       (effects (font (size 1.27 1.27)) hide)
     )
-    (pin "1")
-    (pin "2")
+    (property "manf" "CAMDENBOSS" (id 4) (at 43.18 64.77 0)
+      (effects (font (size 1.27 1.27)) hide)
+    )
+    (property "manf#" "CTBP0108/2" (id 5) (at 43.18 64.77 0)
+      (effects (font (size 1.27 1.27)) hide)
+    )
+    (property "S1MN" "AMPHENOL" (id 6) (at 43.18 64.77 0)
+      (effects (font (size 1.27 1.27)) hide)
+    )
+    (property "S1PN" "VI0221550000G" (id 7) (at 43.18 64.77 0)
+      (effects (font (size 1.27 1.27)) hide)
+    )
+    (pin "1")
+    (pin "2")
+  )
+  (symbol (lib_id "Mechanical:MountingHole") (at 29.845 114.935 0) (unit 1)
+    (in_bom no) (on_board yes) (fields_autoplaced)
+    (property "Reference" "H2" (id 0) (at 32.385 114.1003 0)
+      (effects (font (size 1.27 1.27)) (justify left))
+    )
+    (property "Value" "MountingHole_2.5mm_Pad_TopOnly" (id 1) (at 32.385 116.6372 0)
+      (effects (font (size 1.27 1.27)) (justify left))
+    )
+    (property "Footprint" "MountingHole:MountingHole_2.5mm_Pad_TopOnly" (id 2) (at 29.845 114.935 0)
+      (effects (font (size 1.27 1.27)) hide)
+    )
+    (property "Datasheet" "~" (id 3) (at 29.845 114.935 0)
+      (effects (font (size 1.27 1.27)) hide)
+    )
   )
   (symbol (lib_id "Isolator:PC817") (at 59.69 72.39 270) (unit 1)
@@
     (property "Datasheet" "http://www.soselectronic.cz/a_info/resource/d/pc817.pdf" (id 3) (at 59.69 72.39 0)
       (effects (font (size 1.27 1.27)) (justify left) hide)
+    )
+    (property "manf" "BROADCOM" (id 4) (at 59.69 72.39 0)
+      (effects (font (size 1.27 1.27)) hide)
+    )
+    (property "manf#" "HCPL-817-000E" (id 5) (at 59.69 72.39 0)
+      (effects (font (size 1.27 1.27)) hide)
     )
     (pin "1")
@@
       (effects (font (size 1.27 1.27)) (justify left))
     )
-    (property "Value" "330" (id 1) (at 57.15 57.15 0)
+    (property "Value" "330Ω" (id 1) (at 55.245 57.785 0)
       (effects (font (size 1.27 1.27)) (justify left))
     )
@@
       (effects (font (size 1.27 1.27)) hide)
     )
-    (pin "1")
-    (pin "2")
+    (property "manf" "YAGEO" (id 4) (at 62.23 55.88 0)
+      (effects (font (size 1.27 1.27)) hide)
+    )
+    (property "manf#" "CFR-25JR-52-330R" (id 5) (at 62.23 55.88 0)
+      (effects (font (size 1.27 1.27)) hide)
+    )
+    (pin "1")
+    (pin "2")
+  )
+  (symbol (lib_id "Mechanical:MountingHole") (at 29.845 121.285 0) (unit 1)
+    (in_bom no) (on_board yes) (fields_autoplaced)
+    (property "Reference" "H3" (id 0) (at 32.385 120.4503 0)
+      (effects (font (size 1.27 1.27)) (justify left))
+    )
+    (property "Value" "MountingHole_2.5mm_Pad_TopOnly" (id 1) (at 32.385 122.9872 0)
+      (effects (font (size 1.27 1.27)) (justify left))
+    )
+    (property "Footprint" "MountingHole:MountingHole_2.5mm_Pad_TopOnly" (id 2) (at 29.845 121.285 0)
+      (effects (font (size 1.27 1.27)) hide)
+    )
+    (property "Datasheet" "~" (id 3) (at 29.845 121.285 0)
+      (effects (font (size 1.27 1.27)) hide)
+    )
   )
   (sheet_instances
@@
       (reference "Gazpar1") (unit 1) (value "G-") (footprint "TerminalBlock:TerminalBlock_bornier-2_P5.08mm")
     )
+    (path "/8a11f2c7-a2ec-4e8d-b9e8-7113c6463090"
+      (reference "H1") (unit 1) (value "MountingHole_2.5mm_Pad_TopOnly") (footprint "MountingHole:MountingHole_2.5mm_Pad_TopOnly")
+    )
+    (path "/ce4aadf0-2407-47d8-82a2-42535b56ba29"
+      (reference "H2") (unit 1) (value "MountingHole_2.5mm_Pad_TopOnly") (footprint "MountingHole:MountingHole_2.5mm_Pad_TopOnly")
+    )
+    (path "/f9fdcdbf-c2fd-4043-b7fb-790beec0f544"
+      (reference "H3") (unit 1) (value "MountingHole_2.5mm_Pad_TopOnly") (footprint "MountingHole:MountingHole_2.5mm_Pad_TopOnly")
+    )
+    (path "/32dd8299-2e9a-4bb9-b379-6e0d46d2302b"
+      (reference "H4") (unit 1) (value "MountingHole_2.5mm_Pad_TopOnly") (footprint "MountingHole:MountingHole_2.5mm_Pad_TopOnly")
+    )
     (path "/d66d3c12-11ce-4566-9a45-962e329503d8"
-      (reference "R1") (unit 1) (value "330") (footprint "Resistor_THT:R_Axial_DIN0207_L6.3mm_D2.5mm_P7.62mm_Horizontal")
+      (reference "R1") (unit 1) (value "330Ω") (footprint "Resistor_THT:R_Axial_DIN0207_L6.3mm_D2.5mm_P7.62mm_Horizontal")
     )
     (path "/a8e40a2e-59cf-4d65-ba8c-17cb2e89c54e"
-      (reference "R2") (unit 1) (value "1k") (footprint "Resistor_THT:R_Axial_DIN0207_L6.3mm_D2.5mm_P7.62mm_Horizontal")
+      (reference "R2") (unit 1) (value "1kΩ") (footprint "Resistor_THT:R_Axial_DIN0207_L6.3mm_D2.5mm_P7.62mm_Horizontal")
     )
     (path "/d350f891-7644-4c4e-80f5-20ae02817759"
@@
     )
     (path "/4c8704fa-310a-4c01-8dc1-2b7e2727fea0"
-      (reference "U2") (unit 1) (value "ESP32-DEVKITC-32D") (footprint "MODULE_ESP32-DEVKITC-32D")
-    )
-  )
+      (reference "U2") (unit 1) (value "ESP32-DEVKITC-32D") (footprint "ESP32-DEVKITC-32D:MODULE_ESP32-DEVKITC-32D")
+    )
+  )
